File: tac5212_audio_board_single_ended.kicad_sch (KiCad schematic)
At the start: 112 parts, among them J10 Conn_02x08_Odd_Even, J1002 TAC5212, J2 Conn_02x08_Odd_Even, J3 Conn_02x08_Odd_Even, J4 HEADPHONE, J5 HEADPHONE, J6 Conn_02x08_Odd_Even, J7 Conn_02x08_Odd_Even, J8 Conn_02x08_Odd_Even, J9 Conn_02x08_Odd_Even, U1 Single Buffer - 74LVC1G125GV,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, U2 3.3v LDO - TLV74133PDQNR

Commit message: update
Parts:
- board_outline1: footprint project_fp:audio_module_board_outline_50x34.5_b1 -> project_fp:audio_module_board_outline_50x34.5_c1
Changed lines of the file:
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@@
 			)
 		)
-		(property "Footprint" "project_fp:audio_module_board_outline_50x34.5_b1"
+		(property "Footprint" "project_fp:audio_module_board_outline_50x34.5_c1"
 			(at 247.65 370.84 0)
 			(effects

Commit message: update
Parts:
- removed H1, H2, H3, H4: MountingHole_Pad, MountingHole:MountingHole_2.2mm_M2_DIN965_Pad, symbol Mechanical:MountingHole_Pad
- removed I2C1001: ~, Connector_PinHeader_2.54mm:PinHeader_1x04_P2.54mm_Vertical, symbol Connector:Conn_01x04_Pin
- removed SCL1, SDA1: jumper, project_fp:SolderJumper-3_P1.3mm_Bridged12_Pad1.0x1.5mm_NO_REF, symbol TEENSY_4.0_PCM5242_TPA6120A2-rescue:SolderJumper_3_Bridged12-project_lib
- SCL1001, SDA1001: footprint project_fp:SolderJumper-3_P1.3mm_Bridged12_Pad1.0x1.5mm_NO_REF -> project_fp:jumper_slice; symbol TEENSY_4.0_PCM5242_TPA6120A2-rescue:SolderJumper_3_Bridged12-project_lib -> Jumper:Jumper_2_Bridged
- board_outline1: symbol board_outline:audio_project_board -> Connector_Generic:Conn_02x33_Odd_Even; now in the parts list
Connections:
- net 5212_BCLK1: now also board_outline1.11 (Pin_11)
- net 5212_LRCK1: now also board_outline1.13 (Pin_13)
- net 5212_MCLK1: now also board_outline1.19 (Pin_19)
- net 5212_SCL: now also board_outline1.37 (Pin_37); no longer SCL1001.2 (C)
- net 5212_SCL_A: now also board_outline1.17 (Pin_17)
- net 5212_SDA: now also board_outline1.38 (Pin_38); no longer SDA1001.2 (C)
- net 5212_SDA_A: now also board_outline1.15 (Pin_15)
- net 5V: now also board_outline1.3 (Pin_3)
- net AUX1L: now also board_outline1.26 (Pin_26)
- net AUX1R: now also board_outline1.28 (Pin_28)
- net AUX2L: now also board_outline1.22 (Pin_22)
- net AUX2R: now also board_outline1.24 (Pin_24)
- net DSP_12V: now also board_outline1.5 (Pin_5)
- net DSP_DATA_IN: now also board_outline1.7 (Pin_7)
- net DSP_DATA_OUT: now also board_outline1.9 (Pin_9)
- net DSP_HELD_HIGH: now also board_outline1.1 (Pin_1)
- net GNDD: now also board_outline1.10 (Pin_10), board_outline1.12 (Pin_12), board_outline1.14 (Pin_14), board_outline1.16 (Pin_16), board_outline1.18 (Pin_18), board_outline1.2 (Pin_2), board_outline1.20 (Pin_20), board_outline1.4 (Pin_4), board_outline1.44 (Pin_44), board_outline1.6 (Pin_6), board_outline1.8 (Pin_8); no longer board_outline1.1 (GND)
- net PHONE1L: now also board_outline1.30 (Pin_30)
- net PHONE1R: now also board_outline1.32 (Pin_32)
- net RCAL: now also board_outline1.34 (Pin_34)
- net RCAR: now also board_outline1.36 (Pin_36)
- net GPO1: now reaches GPIO1001.3 (Pin_3), R1006.1
- net GPO1: now also board_outline1.41 (Pin_41)
- net MICBIAS: now reaches C1008.1, GPIO1001.1 (Pin_1), J1002.14 (MICBIAS)
- net MICBIAS: now also board_outline1.43 (Pin_43)
- net GPIO2: now reaches GPIO1001.4 (Pin_4), R1007.1
- net GPIO2: now also board_outline1.40 (Pin_40)
- net GPI1: now reaches GPIO1001.2 (Pin_2), R1005.1
- net GPI1: now also board_outline1.42 (Pin_42)
- net GPIO1: now reaches GPIO1001.5 (Pin_5), R1008.1
- net GPIO1: now also board_outline1.39 (Pin_39)
Other:
- note removed: "I2C/i2S BYPASS"
- moved on the sheet: C1008, GPIO1001, R1005, R1006, R1007, R1008

Commit message: UPDATE
Parts:
- added MCLK1: jumper, project_fp:jumper_slice, symbol Jumper:Jumper_2_Bridged
Connections:
- net DSP_DATA_IN is gone; now on net 5212_DOUT1+: XIA1.7 (DSP_DATA_IN), XIA2.4 (Pin_4), board_outline1.7 (Pin_7)
- net DSP_DATA_OUT is gone; now on net 5212_DIN1: XIA1.9 (DSP_DATA_OUT), XIA2.5 (Pin_5), board_outline1.9 (Pin_9)
- net 5212_MCLK1: now also MCLK1.2 (B)
- net GNDD: now also board_outline1.39 (Pin_39); no longer board_outline1.44 (Pin_44)
- net GPI1: now also board_outline1.43 (Pin_43), MCLK1.1 (A); no longer board_outline1.42 (Pin_42)
- net GPIO1: now also board_outline1.40 (Pin_40); no longer board_outline1.39 (Pin_39)
- net GPIO2: now also board_outline1.41 (Pin_41); no longer board_outline1.40 (Pin_40)
- net GPO1: now also board_outline1.42 (Pin_42); no longer board_outline1.41 (Pin_41)
- net MICBIAS: now also board_outline1.44 (Pin_44); no longer board_outline1.43 (Pin_43)
Changed lines of the file:
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@@
 	)
 	(junction
+		(at 68.58 83.82)
+		(diameter 0)
+		(color 0 0 0 0)
+	)
+	(junction
 		(at 58.42 55.88)
 		(diameter 0)
@@
 	(wire
 		(pts
-			(xy 52.07 83.82) (xy 81.28 83.82)
+			(xy 52.07 83.82) (xy 68.58 83.82)
 		)
 		(stroke
@@
 	(wire
 		(pts
+			(xy 66.04 100.33) (xy 68.58 100.33)
+		)
+		(stroke
+			(width 0)
+			(type default)
+		)
+	)
+	(wire
+		(pts
 			(xy 205.74 316.23) (xy 231.14 316.23)
 		)
@@
 	(wire
 		(pts
+			(xy 68.58 100.33) (xy 68.58 83.82)
+		)
+		(stroke
+			(width 0)
+			(type default)
+		)
+	)
+	(wire
+		(pts
 			(xy 248.92 533.4) (xy 250.19 533.4)
 		)
@@
 	(wire
 		(pts
-			(xy 255.27 369.57) (xy 243.84 369.57)
+			(xy 219.71 364.49) (xy 231.14 364.49)
 		)
 		(stroke
@@
 	(wire
 		(pts
+			(xy 68.58 83.82) (xy 81.28 83.82)
+		)
+		(stroke
+			(width 0)
+			(type default)
+		)
+	)
+	(wire
+		(pts
 			(xy 86.36 83.82) (xy 92.71 83.82)
 		)
@@
 	)
 	(label "MICBIAS"
-		(at 231.14 369.57 180)
+		(at 243.84 369.57 0)
 		(fields_autoplaced yes)
 		(effects
@@
 				(size 1.27 1.27)
 			)
-			(justify right bottom)
+			(justify left bottom)
 		)
 	)
@@
 	)
 	(label "GPIO1"
-		(at 231.14 364.49 180)
+		(at 243.84 364.49 0)
 		(fields_autoplaced yes)
 		(effects
@@
 				(size 1.27 1.27)
 			)
-			(justify right bottom)
+			(justify left bottom)
 		)
 	)
@@
 	)
 	(label "GPO1"
-		(at 231.14 367.03 180)
+		(at 243.84 367.03 0)
 		(fields_autoplaced yes)
 		(effects
@@
 				(size 1.27 1.27)
 			)
-			(justify right bottom)
+			(justify left bottom)
 		)
 	)
@@
 	)
 	(label "GPIO2"
-		(at 243.84 364.49 0)
+		(at 231.14 367.03 180)
 		(fields_autoplaced yes)
 		(effects
@@
 				(size 1.27 1.27)
 			)
-			(justify left bottom)
+			(justify right bottom)
 		)
 	)
@@
 	)
 	(label "GPI1"
-		(at 243.84 367.03 0)
+		(at 231.14 369.57 180)
 		(fields_autoplaced yes)
 		(effects
@@
 				(size 1.27 1.27)
 			)
-			(justify left bottom)
+			(justify right bottom)
 		)
 	)
@@
 		)
 	)
-	(global_label "DSP_DATA_IN"
-		(shape input)
-		(at 205.74 323.85 180)
-		(fields_autoplaced yes)
-		(effects
-			(font
-				(size 0.8 0.8)
-			)
-			(justify right)
-		)
-		(property "Intersheetrefs" "${INTERSHEET_REFS}"
-			(at 196.2788 323.85 0)
-			(effects
-				(font
-					(size 1.27 1.27)
-				)
-				(justify right)
-				(hide yes)
-			)
-		)
-	)
 	(global_label "5V"
 		(shape input)
@@
 		)
 	)
-	(global_label "DSP_DATA_OUT"
-		(shape input)
-		(at 205.74 326.39 180)
-		(fields_autoplaced yes)
-		(effects
-			(font
-				(size 0.8 0.8)
-			)
-			(justify right)
-		)
-		(property "Intersheetrefs" "${INTERSHEET_REFS}"
-			(at 195.2122 326.39 0)
-			(effects
-				(font
-					(size 1.27 1.27)
-				)
-				(justify right)
-				(hide yes)
-			)
-		)
-	)
 	(global_label "OUT2P"
 		(shape input)
@@
 		)
 	)
+	(global_label "5212_DOUT1+"
+		(shape input)
+		(at 205.74 323.85 180)
+		(fields_autoplaced yes)
+		(effects
+			(font
+				(size 0.8 0.8)
+			)
+			(justify right)
+		)
+		(property "Intersheetrefs" "${INTERSHEET_REFS}"
+			(at 195.3645 323.85 0)
+			(effects
+				(font
+					(size 1.27 1.27)
+				)
+				(justify right)
+				(hide yes)
+			)
+		)
+	)
 	(global_label "AUX1R"
 		(shape input)
@@
 		)
 	)
+	(global_label "5212_DIN1"
+		(shape input)
+		(at 205.74 326.39 180)
+		(fields_autoplaced yes)
+		(effects
+			(font
+				(size 0.8 0.8)
+			)
+			(justify right)
+		)
+		(property "Intersheetrefs" "${INTERSHEET_REFS}"
+			(at 197.4216 326.39 0)
+			(effects
+				(font
+					(size 1.27 1.27)
+				)
+				(justify right)
+				(hide yes)
+			)
+		)
+	)
 	(global_label "AUX1L"
 		(shape input)
@@
 		)
 	)
+	(global_label "5212_MCLK1"
+		(shape input)
+		(at 55.88 100.33 180)
+		(fields_autoplaced yes)
+		(effects
+			(font
+				(size 1.27 1.27)
+			)
+			(justify right)
+		)
+		(property "Intersheetrefs" "${INTERSHEET_REFS}"
+			(at 40.8602 100.33 0)
+			(effects
+				(font
+					(size 1.27 1.27)
+				)
+				(justify right)
+				(hide yes)
+			)
+		)
+	)
 	(global_label "OUT1P"
 		(shape input)
@@
 	)
 	(symbol
+		(lib_id "Jumper:Jumper_2_Bridged")
+		(at 60.96 100.33 180)
+		(unit 1)
+		(exclude_from_sim yes)
+		(in_bom yes)
+		(on_board yes)
+		(dnp no)
+		(property "Reference" "MCLK1"
+			(at 60.96 105.537 0)
+			(effects
+				(font
+					(size 1.27 1.27)
+				)
+			)
+		)
+		(property "Value" "jumper"
+			(at 60.96 103.2256 0)
+			(effects
+				(font
+					(size 1.27 1.27)
+				)
+			)
+		)
+		(property "Footprint" "project_fp:jumper_slice"
+			(at 60.96 100.33 0)
+			(effects
+				(font
+					(size 1.27 1.27)
+				)
+				(hide yes)
+			)
+		)
+		(property "Datasheet" "~"
+			(at 60.96 100.33 0)
+			(effects
+				(font
+					(size 1.27 1.27)
+				)
+				(hide yes)
+			)
+		)
+		(property "Description" "Jumper, 2-pole, closed/bridged"
+			(at 60.96 100.33 0)
+			(effects
+				(font
+					(size 1.27 1.27)
+				)
+				(hide yes)
+			)
+		)
+		(property "PCBWAY_2020_04_18" "NO COMPONENT"
+			(at 60.96 100.33 0)
+			(effects
+				(font
+					(size 1.27 1.27)
+				)
+				(hide yes)
+			)
+		)
+		(property "PCBWAY_2020-06-09" "NO COMPONENT"
+			(at 60.96 100.33 0)
+			(effects
+				(font
+					(size 1.27 1.27)
+				)
+				(hide yes)
+			)
+		)
+		(property "PCBWAY_2020-08-27" "NO COMPONENT"
+			(at 60.96 100.33 0)
+			(effects
+				(font
+					(size 1.27 1.27)
+				)
+				(hide yes)
+			)
+		)
+		(pin "1"
+		)
+		(pin "2"
+		)
+		(instances
+			(project "tac5212_audio_board_single_ended"
+				(path "/8cee3af6-3893-45a9-89a4-21657973eeff"
+					(reference "MCLK1")
+					(unit 1)
+				)
+			)
+		)
+	)
+	(symbol
 		(lib_id "Device:R_Small")
 		(at 83.82 88.9 90)
@@
 	(symbol
 		(lib_id "power:GNDD")
-		(at 255.27 369.57 0)
+		(at 219.71 364.49 0)
 		(unit 1)
 		(exclude_from_sim no)
@@
 		(dnp no)
 		(property "Reference" "#PWR011"
-			(at 255.27 375.92 0)
+			(at 219.71 370.84 0)
 			(effects
 				(font
@@
 		)
 		(property "Value" "GNDD"
-			(at 255.27 385.572 0)
+			(at 219.71 380.492 0)
 			(effects
 				(font
@@
 		)
 		(property "Footprint" ""
-			(at 255.27 369.57 0)
+			(at 219.71 364.49 0)
 			(effects
 				(font
@@
 		)
 		(property "Datasheet" ""
-			(at 255.27 369.57 0)
+			(at 219.71 364.49 0)
 			(effects
 				(font
@@
 		)
 		(property "Description" ""
-			(at 255.27 369.57 0)
+			(at 219.71 364.49 0)
 			(effects
 				(font
