File: tac5212_audio_board_single_ended.kicad_pcb (KiCad board)
At the start: 4 copper layers, 42 x 26.5 mm, 110 parts, among them T108 Tab, T109 Tab, T110 Tab, T111 Tab, U108 Single Buffer with Tri-state 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, U109 3.3v LDO - TLV74133PDBVR

Commit message: update
Parts:
- moved C131 1.60 mm to (93.2, 120.0)
Routing:
- net GNDD: track 122.0 -> 128.8 mm
- net 3.3v_IDE: track 50.6 -> 47.5 mm
- net 5V: track 30.0 -> 29.3 mm
- net Earth: track 309.2 -> 309.0 mm, vias 10 -> 9

Commit message: update
Parts:
- C128: value 1uF -> 0.1uF; footprint project_fp:C_0603_1608Metric_Pad1.08x0.95mm_HandSolder -> project_fp:C_0402_1005Metric
- C131: value 47uF -> 10uF
- U108: footprint project_fp:SOT-23-5 -> Package_TO_SOT_SMD:SOT-353_SC-70-5
- moved INP2 0.79 mm to (121.5, 105.5)
- moved INM1 0.50 mm to (119.0, 106.5)
- moved C130 0.32 mm to (93.1, 120.3)
Routing:
- net GNDD: track 128.8 -> 167.6 mm
- net Earth: track 309.0 -> 295.5 mm, vias 9 -> 8
- net 5V: track 29.3 -> 28.4 mm
