File: t-dsp_tac5212_pro_audio_module.kicad_sch (KiCad schematic)
At the start: 119 parts, among them J3V108 jumper, J5V108 jumper, T108 Tab, T109 Tab, T110 Tab, T111 Tab, U108 Single Buffer with Tri-state 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, U109 3.3v LDO - TLV74133PDBVR

Commit message: Fix Package field conflicts and enable gerber job file
- C128: Package C0603 → C0402 (matches footprint)
- C124: Package C0805 → C0603 (matches footprint)
- Enable gerber job file for automatic layer identification by fabs
Parts:
- C124: Package / Case C0805 -> C0603
- C128: Package / Case C0603 -> C0402
Changed lines of the file:
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@@
 			)
 		)
-		(property "Package / Case" "C0603"
+		(property "Package / Case" "C0402"
 			(at 189.23 273.05 0)
 			(effects
@@
 			)
 		)
-		(property "Package / Case" "C0805"
+		(property "Package / Case" "C0603"
 			(at 468.63 293.37 0)
 			(effects
