File: t-dsp_tac5212_pro_audio_module.kicad_sch (KiCad schematic)
At the start: 119 parts, among them J3V108 jumper, J5V108 jumper, T108 Tab, T109 Tab, T110 Tab, T111 Tab, U108 Single Buffer with Tri-state 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, U109 3.3v LDO - TLV74133PDBVR

Commit message: Add schematic and PCB layout PDFs to manufacturing output
Co-Authored-By: Claude Opus 4.6 <noreply@anthropic.com>
Other:
- note added: "PANEL TABS"
- moved on the sheet: ADD108, ADD110, ADD111, ADD112, C108, C109, C110, C111, C112, C113, C114, C115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
