File: t-dsp_tac5212_pro_audio_module.kicad_sch (KiCad schematic)
At the start: 119 parts, among them J3V108 jumper, J5V108 jumper, T108 Tab, T109 Tab, T110 Tab, T111 Tab, U108 Single Buffer with Tri-state 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, U109 3.3v LDO - TLV74133PDBVR

Commit message: Add 3D renders, hide ref designators, fix legacy 3D model paths
- Add Blender 3D render output (8 views: top, bottom, 4 sides, 2 isometric)
  to KiBot config and manufacturing ZIP
- Split CI workflow into 3 steps: manufacturing outputs, 3D renders
  (kicad9_auto_full), and ZIP packaging
- Add PCB spec report to manufacturing outputs
- Hide reference designators and component values from silkscreen
- Replace legacy ${KISYS3DMOD} with ${KICAD9_3DMODEL_DIR} across all
  footprint libraries and PCB (47 files)
- Add new 3D models (TPD1E10B06, VQFN-24) and footprints
- Set net tie footprint type on jumper components

Co-Authored-By: Claude Opus 4.6 <noreply@anthropic.com>
Parts:
- C113, C114, C120, C122: footprint Capacitor_SMD:C_0603_1608Metric_Pad1.08x0.95mm_HandSolder -> project_fp:C_0603_1608Metric_Pad1.08x0.95mm_HandSolder
- G119: footprint project_fp:jumper_slice_alt1 -> project_fp:jumper_slice
- GND108: Label GND -> G
- MCLK108: footprint Jumper:SolderJumper-2_P1.3mm_Open_Pad1.0x1.5mm -> project_fp:SolderJumper-2_P1.3mm_Open_Pad1.0x1.5mm_Master_Clock
- T108, T109, T110, T111: footprint kikit:Tab -> project_fp:Tab
- TAC108-Q1: footprint Package_DFN_QFN:Texas_RHB0032E_VQFN-32-1EP_5x5mm_P0.5mm_EP3.45x3.45mm_ThermalVias -> project_fp:Texas_RHB0032E_VQFN-32-1EP_5x5mm_P0.5mm_EP3.45x3.45mm_ThermalVias
- U108: footprint Package_TO_SOT_SMD:SOT-353_SC-70-5 -> project_fp:SOT-353_SC-70-5
Connections:
- net Earth: now also E109.2, G119.2, GND108.2; no longer E109.1, G119.1, GND108.1
- net GNDD: now also GND108.1; no longer GND108.2
- net at T*C108.2, T*C109.2, T*C110.2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: now also G119.1; no longer G119.2
- net at board_outline108.50 (AGND): now also E109.1; no longer E109.2
Other:
- moved on the sheet: E109, G119, GND108
Changed lines of the file:
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@@
 			)
 		)
-		(property "Footprint" "kikit:Tab"
+		(property "Footprint" "project_fp:Tab"
 			(at 107.95 595.63 0)
 			(effects
@@
 			)
 		)
-		(property "Footprint" "Package_TO_SOT_SMD:SOT-353_SC-70-5"
+		(property "Footprint" "project_fp:SOT-353_SC-70-5"
 			(at 133.35 457.2 0)
 			(effects
@@
 			)
 		)
-		(property "Footprint" "kikit:Tab"
+		(property "Footprint" "project_fp:Tab"
 			(at 152.4 595.63 0)
 			(effects
@@
 			)
 		)
-		(property "Footprint" "kikit:Tab"
+		(property "Footprint" "project_fp:Tab"
 			(at 128.27 596.9 0)
 			(effects
@@
 			)
 		)
-		(property "Footprint" "Jumper:SolderJumper-2_P1.3mm_Open_Pad1.0x1.5mm"
+		(property "Footprint" "project_fp:SolderJumper-2_P1.3mm_Open_Pad1.0x1.5mm_Master_Clock"
 			(at 111.76 132.08 0)
 			(effects
@@
 			)
 		)
-		(property "Footprint" "Package_DFN_QFN:Texas_RHB0032E_VQFN-32-1EP_5x5mm_P0.5mm_EP3.45x3.45mm_ThermalVias"
+		(property "Footprint" "project_fp:Texas_RHB0032E_VQFN-32-1EP_5x5mm_P0.5mm_EP3.45x3.45mm_ThermalVias"
 			(at 182.88 119.38 0)
 			(effects
@@
 			)
 		)
-		(property "Footprint" "kikit:Tab"
+		(property "Footprint" "project_fp:Tab"
 			(at 176.53 595.63 0)
 			(effects
@@
 			)
 		)
-		(property "Footprint" "Capacitor_SMD:C_0603_1608Metric_Pad1.08x0.95mm_HandSolder"
+		(property "Footprint" "project_fp:C_0603_1608Metric_Pad1.08x0.95mm_HandSolder"
 			(at 429.26 170.18 0)
 			(effects
@@
 	(symbol
 		(lib_id "proejct_lib:NetTie_2")
-		(at 190.5 292.1 180)
+		(at 190.5 292.1 0)
 		(unit 1)
 		(exclude_from_sim no)
@@
 		(dnp yes)
 		(property "Reference" "E109"
-			(at 185.166 295.656 0)
+			(at 195.834 288.544 0)
 			(effects
 				(font
@@
 		)
 		(property "Value" "jumper"
-			(at 196.85 295.91 0)
+			(at 184.15 288.29 0)
 			(effects
 				(font
@@
 			)
 		)
-		(property "Footprint" "Capacitor_SMD:C_0603_1608Metric_Pad1.08x0.95mm_HandSolder"
+		(property "Footprint" "project_fp:C_0603_1608Metric_Pad1.08x0.95mm_HandSolder"
 			(at 430.53 201.93 0)
 			(effects
@@
 			)
 		)
-		(property "Footprint" "Capacitor_SMD:C_0603_1608Metric_Pad1.08x0.95mm_HandSolder"
+		(property "Footprint" "project_fp:C_0603_1608Metric_Pad1.08x0.95mm_HandSolder"
 			(at 429.26 271.78 0)
 			(effects
@@
 	(symbol
 		(lib_id "proejct_lib:NetTie_2")
-		(at 231.14 189.23 180)
+		(at 231.14 189.23 0)
 		(unit 1)
 		(exclude_from_sim no)
@@
 		(dnp yes)
 		(property "Reference" "GND108"
-			(at 231.14 191.262 0)
+			(at 231.14 187.198 0)
 			(effects
 				(font
@@
 		)
 		(property "Value" "BRIDGE"
-			(at 231.14 187.198 0)
+			(at 231.14 191.262 0)
 			(effects
 				(font
@@
 			)
 		)
-		(property "Label" "GND"
+		(property "Label" "G"
 			(at 231.14 189.23 0)
 			(effects
@@
 			)
 		)
-		(property "Footprint" "Capacitor_SMD:C_0603_1608Metric_Pad1.08x0.95mm_HandSolder"
+		(property "Footprint" "project_fp:C_0603_1608Metric_Pad1.08x0.95mm_HandSolder"
 			(at 433.07 236.22 0)
 			(effects
@@
 	(symbol
 		(lib_id "proejct_lib:NetTie_2")
-		(at 154.94 382.27 90)
+		(at 154.94 382.27 270)
 		(unit 1)
 		(exclude_from_sim no)
@@
 		(dnp yes)
 		(property "Reference" "G119"
-			(at 153.924 376.936 0)
+			(at 155.956 387.604 0)
 			(effects
 				(font
@@
 		)
 		(property "Value" "jumper"
-			(at 153.67 388.62 0)
+			(at 156.21 375.92 0)
 			(effects
 				(font
@@
 			)
 		)
-		(property "Footprint" "project_fp:jumper_slice_alt1"
+		(property "Footprint" "project_fp:jumper_slice"
 			(at 154.94 382.27 0)
 			(effects
